File: taito_video_processor_pcb/taito_video_processor_pcb.sch (KiCad schematic (older format))
At the start: 12 parts, among them J3 50pin, U18 68A45, U19 86_2, U20 86_1, U34 LS374, U50 86_3, U51 LS86

Commit message: Continued the schematic layout.
Parts:
- added BT1: 3.6V, symbol Device:Battery
- added C101, C22, C42, C44, C45, C9: 10uf, symbol Device:CP1
- added C65: 470pf, symbol Device:C
- added FB7: Ferrite_Bead, symbol Device:Ferrite_Bead
- added J19: 2pin, symbol taito_pcb:2pin
- added J6: 50pin, symbol taito_pcb:50pin
- added JB2: W1, symbol Device:Jumper
- added LED1, LED2, LED3, LED4, LED5, LED6: LED, symbol Device:LED
- added Q8: 2N3905, symbol Device:Q_PNP_EBC
- added R1, R10, R51, R52, R53, R54, R55, R56, R57, R58: 33, symbol Device:R_US
- added R38, R6, R62, R66, R68, R69: 3.3k, symbol Device:R_US
- added R39, R40, R41, R42, R43, R44: 330, symbol Device:R_US
- added R61: 390, symbol Device:R_US
- added R64: 120, symbol Device:R_US
- added R65: 150, symbol Device:R_US
- added U10, U11, U12, U13, U14, U15, U16, U17, U26, U27, U28, U29, U30, U31, U32, U33: 4116, symbol taito_pcb:4116
- added U100, U103: LS00, symbol Asteroids:LS00
- added U101: LS08, symbol Asteroids:LS08
- added U102: LS10, symbol Asteroids:LS10
- added U35, U52, U53, U54: 153_1, symbol taito_pcb:153_1
- added U39: LS04, symbol Asteroids:LS04
- added U40: 7417, symbol taito_pcb:7417
- added U49, U88: LS32, symbol Asteroids:LS32
- added unit 3 of U51
- added unit 2 of U51
- added U72: LS374, symbol Asteroids:LS374
- added U77, U78: 373, symbol taito_pcb:373
- added U? (x2): 6514_1, symbol taito_pcb:6514_1
Connections:
- net VAQ is gone; now on net VA0: U18.24 (RS)
- net +5V: now also C45.1, LED1.2 (A), LED2.2 (A), LED3.2 (A), LED4.2 (A), LED5.2 (A), LED6.2 (A), Q8.1 (E), R38.1, R6.1, R62.1, R66.1, R68.1, R69.1, U10.9, U101.14 (VCC), U102.14 (VCC), U103.14 (VCC), U11.9, U12.9, U13.9, U14.9, U15.9, U16.9, U17.9, U26.9, U27.9, U28.9, U29.9, U30.9, U31.9, U32.9, U33.9, U35.16 (VCC), U49.14 (VCC), U52.16 (VCC), U53.16 (VCC), U54.16 (VCC), U72.20 (VCC), U77.20 (VCC), U78.20 (VCC), U88.14 (VCC)
- net GND: now also C101.2, C22.2, C42.2, C44.1, C45.2, C65.2, C9.1, J19.1, J6.10, J6.12, J6.24, J6.26, J6.28, J6.29, J6.44, J6.46, JB2.2, U10.16, U100.1, U100.10, U100.2, U100.4, U100.5, U100.7 (GND), U100.9, U101.7 (GND), U102.7 (GND), U103.7 (GND), U11.16, U12.16, U13.16, U14.16, U15.16, U16.16, U17.16, U26.16, U27.16, U28.16, U29.16, U30.16, U31.16, U32.16, U33.16, U35.1, U35.15, U35.8 (GND), U49.7 (GND), U51.9, U52.1, U52.15, U52.8 (GND), U53.1, U53.15, U53.8 (GND), U54.1, U54.15, U54.8 (GND), U72.1 (OE), U72.10 (GND), U77.10 (GND), U78.10 (GND), U88.7 (GND), U?.9 (GND), U?.9 (GND)
- net M0: now also U10.5, U11.5, U12.5, U13.5, U14.5, U15.5, U16.5, U17.5, U26.5, U27.5, U28.5, U29.5, U30.5, U31.5, U32.5, U33.5, U54.7
- net M1: now also U10.6, U11.6, U12.6, U13.6, U14.6, U15.6, U16.6, U17.6, U26.6, U27.6, U28.6, U29.6, U30.6, U31.6, U32.6, U33.6, U53.9
- net M2: now also U10.7, U11.7, U12.7, U13.7, U14.7, U15.7, U16.7, U17.7, U26.7, U27.7, U28.7, U29.7, U30.7, U31.7, U32.7, U33.7, U53.7
- net M3: now also U10.12, U11.12, U12.12, U13.12, U14.12, U15.12, U16.12, U17.12, U26.12, U27.12, U28.12, U29.12, U30.12, U31.12, U32.12, U33.12, U35.9
- net M4: now also U10.11, U11.11, U12.11, U13.11, U14.11, U15.11, U16.11, U17.11, U26.11, U27.11, U28.11, U29.11, U30.11, U31.11, U32.11, U33.11, U35.7
- net M5: now also U10.10, U11.10, U12.10, U13.10, U14.10, U15.10, U16.10, U17.10, U26.10, U27.10, U28.10, U29.10, U30.10, U31.10, U32.10, U33.10, U52.9
- net M6: now also U10.13, U11.13, U12.13, U13.13, U14.13, U15.13, U16.13, U17.13, U26.13, U27.13, U28.13, U29.13, U30.13, U31.13, U32.13, U33.13, U52.7
- net VA0: now also U?.5, U?.5
- net VA1: now also U?.6, U?.6
- net VA2: now also U?.7, U?.7
- net VA3: now also U?.4, U?.4
- net VA4: now also U?.3, U?.3
- net VA5: now also U?.2, U?.2
- net VA6: now also U?.1, U?.1
- net VA7: now also U?.17, U?.17
- net VA8: now also U102.2, U?.16, U?.16
- net VA9: now also U102.1, U?.15, U?.15
- net VD0: now also R58.2, U72.18 (D7), U77.19, U78.19, U?.14
- net VD1: now also R57.2, U72.17 (D6), U77.16, U78.16, U?.13
- net VD2: now also R56.2, U72.14 (D5), U77.15, U78.15, U?.12
- net VD3: now also R55.2, U72.13 (D4), U77.12, U78.12, U?.11
- net VD4: now also R54.2, U72.8 (D3), U77.9, U78.9, U?.14
- net VD5: now also R53.2, U72.7 (D2), U77.6, U78.6, U?.13
- net VD6: now also R52.2, U72.4 (D1), U77.5, U78.5, U?.12
- net VD7: now also R51.2, U72.3 (D0), U77.2, U78.2, U?.11
- net VEN: now also U101.5
- net VEQ: now also U103.2
- net X0: now also U53.13
- net X1: now also U53.3
- net X10: now also U35.4
- net X11: now also U52.12
- net X12: now also U52.4
- net X2: now also U35.13
- net X3: now also U35.3
- net X4: now also U52.13
- net X5: now also U52.3
- net X6: now also U54.4
- net X7: now also U53.12
- net X8: now also U53.4
- net X9: now also U35.12
- net ~CAS: now also U10.15, U11.15, U12.15, U13.15, U14.15, U15.15, U16.15, U17.15, U26.15, U27.15, U28.15, U29.15, U30.15, U31.15, U32.15, U33.15
- net ~MRST: now also U100.13
- net ~RAS: now also U10.4, U11.4, U12.4, U13.4, U14.4, U15.4, U16.4, U17.4, U26.4, U27.4, U28.4, U29.4, U30.4, U31.4, U32.4, U33.4
- net at U19.10, U19.13, U19.2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: now also U51.8
- net at U50.10, U50.13, U50.2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: now also U51.2, U51.10, U51.6
- net at U34.11 (Cp): now also U101.6
- new net: R38.2, U51.4
- new net: U100.11, U?.10 (R/~w), U?.10 (R/~w)
- new net: R61.2, U40.12, U?.8 (~CS), U?.8 (~CS)
- new net: U100.12, U101.3
- new net: Q8.2 (B), R65.1
- new net: U101.2, U102.12
- new net: FB7.1, R66.2, U102.13
- new net: U103.1, U39.8
- new net: U103.3, U40.13
- new net: BT1.1 (+), R64.1, R65.2
- new net: BT1.2 (-), JB2.1
- new net: C65.1, FB7.2, J19.2
- new net: U72.11 (Cp), U88.3
- new net: R41.2, U72.12 (O4)
- new net: R42.2, U72.15 (O5)
- new net: R39.2, U72.2 (O0)
- new net: R44.2, U72.5 (O1)
- new net: R40.2, U72.6 (O2)
- new net: R43.2, U72.9 (O3)
- new net: LED1.1 (K), R39.1
- new net: LED3.1 (K), R44.1
- new net: LED2.1 (K), R40.1
- new net: LED4.1 (K), R43.1
- new net: LED6.1 (K), R41.1
- new net: LED5.1 (K), R42.1
- new net: R1.1, U10.3, U11.3, U12.3, U13.3, U14.3, U15.3, U16.3, U17.3
- new net: U49.8, U77.1 (~OE)
- new net: R1.2, U49.6
- new net: R10.1, U26.3, U27.3, U28.3, U29.3, U30.3, U31.3, U32.3, U33.3
- new net: U49.11, U78.1 (~OE)
- new net: R10.2, U49.3
- new net +12V: C22.1, C42.1, U10.8, U11.8, U12.8, U13.8, U14.8, U15.8, U16.8, U17.8, U26.8, U27.8, U28.8, U29.8, U30.8, U31.8, U32.8, U33.8
- new net -5V: C44.2, C9.2, U10.1, U11.1, U12.1, U13.1, U14.1, U15.1, U16.1, U17.1, U26.1, U27.1, U28.1, U29.1, U30.1, U31.1, U32.1, U33.1
- new net BD0: R58.1, U17.2, U33.2
- new net BD1: R57.1, U16.2, U32.2
- new net BD2: R56.1, U15.2, U31.2
- new net BD3: R55.1, U14.2, U30.2
- new net BD4: R54.1, U13.2, U29.2
- new net BD5: R53.1, U12.2, U28.2
- new net BD6: R52.1, U11.2, U27.2
- new net BD7: R51.1, U10.2, U26.2
- new net BPWR: C101.1, Q8.3 (C), R61.1, R64.2, U100.14 (VCC), U?.18 (VCC), U?.18 (VCC)
- new net CR8: U72.19 (O7)
- new net CR9: U72.16 (O6)
- new net DA0: J6.35
- new net DA1: J6.38
- new net DA2: J6.50
- new net DA3: J6.49
- new net DA4: J6.48
- new net DA5: J6.47
- new net DA6: J6.36
- new net DA7: J6.45
- new net DA8: J6.37
- new net DA9: J6.40
- new net DD0: J6.1
- new net DD1: J6.4
- new net DD2: J6.3
- new net DD3: J6.6
- new net DD4: J6.5
- new net DD5: J6.8
- new net DD6: J6.7
- new net DD7: J6.9
- new net DRW: J6.2
- new net INV: J6.42
- new net LA10: U53.10
- new net LA11: U53.6
- new net LA12: U35.10
- new net LA13: U35.6
- new net LA14: U52.10
- new net LA15: U52.6
- new net LA2: U54.5
- new net LA3: U53.11
- new net LA4: U53.5
- new net LA5: U35.11
- new net LA6: U35.5
- new net LA7: U52.11
- new net LA8: U52.5
- new net LA9: U54.6
- new net Q: J6.11
- new net QX: U77.11 (C), U78.11 (C)
- new net R0: U33.14, U78.18
- new net R1: U32.14, U78.17
- new net R10: U15.14, U77.14
- new net R11: U14.14, U77.13
- new net R12: U13.14, U77.8
- new net R13: U12.14, U77.7
- new net R14: U11.14, U77.4
- new net R15: U10.14, U77.3
- new net R2: U31.14, U78.14
- new net R3: U30.14, U78.13
- new net R4: U29.14, U78.8
- new net R5: U28.14, U78.7
- new net R6: U27.14, U78.4
- new net R7: U26.14, U78.3
- new net R8: U17.14, U77.18
- new net R9: U16.14, U77.17
- new net RP6: R6.2
- new net RP62: R62.2
- new net RP68: R68.2
- new net RP69: R69.2
- new net _VS: J6.30
- new net vEQ: U101.4
- new net ~CCLK: U54.3
- new net ~DEIRQ: J6.43
- new net ~DS1: J6.27
- new net ~DS3: J6.31
- new net ~EVEN0: U49.13, U49.2
- new net ~INV: U51.5
- new net ~MUX: U35.14, U52.14, U53.14, U54.14
- new net ~ODD0: U49.10, U49.5
- new net ~QRW: U88.2
- new net ~QX: J6.25, U35.2, U52.2, U53.2, U54.2
- new net ~VEW: U49.1, U49.4
- new net ~VRW: U101.1, U49.12, U49.9
- new net ~VS2: U88.1
- new net ~VSI: U39.9
- no-connect marks 13 -> 37
Other:
- moved on the sheet: RP1, RP2, RP3, RP4, RP5, U18, U19, U20, U34, U50, U51A

Commit message: Continued with the schematic layout.
Parts:
- added C14, C31: 100pf, symbol Device:C
- added R2: 1.5k, symbol Device:R_US
- added R37, R50, R59: 47k, symbol Device:R_US
- added R60, R67: 3.3k, symbol Device:R_US
- added R63: 1k, symbol Device:R_US
- added R7: 220, symbol Device:R_US
- added R8: 2.2k, symbol Device:R_US
- added SW1: SW_Push, symbol Switch:SW_Push
- added TP2: 10MHz, symbol Connector:TestPoint
- added TP3, TP4, TP5, TP6, TP7, TP8: TestPoint, symbol Connector:TestPoint
- added U1, U2, U69: 245_1, symbol taito_pcb:245_1
- added unit 3 of U101
- added U21, U5, U6: 157_1, symbol taito_pcb:157_1
- added U22, U9: LS32, symbol Asteroids:LS32
- added U23: 161_1, symbol taito_pcb:161_1
- added U24, U90: LS04, symbol Asteroids:LS04
- added U25, U70, U71: 374_1, symbol taito_pcb:374_1
- added U3, U4: 2114, symbol Asteroids:2114
- added U36, U89: LS74, symbol Asteroids:LS74
- added U37: LS08, symbol Asteroids:LS08
- added U38: 74S113, symbol taito_pcb:74S113
- added unit 1 of U39
- added unit 2 of U39
- added unit 3 of U39
- added U68, U83, U84: 244_2, symbol taito_pcb:244_2
- added U82: 68A09E, symbol taito_pcb:68A09E
- added unit 4 of U88
- added U97, U98: 244_1, symbol taito_pcb:244_1
- added U99: 138_1, symbol taito_pcb:138_1
- added Y1: Crystal, symbol Device:Crystal
- gave numbers to parts that had none: 2
Connections:
- net +5V: now also R50.1, R59.2, R60.1, R63.2, R67.1, U1.20 (VCC), U2.20 (VCC), U21.16 (VCC), U22.14 (VCC), U23.16 (VCC), U24.14 (VCC), U25.20 (VCC), U3.18 (VSS), U36.14 (VCC), U37.14 (VCC), U38.14 (VCC), U39.14 (VCC), U4.18 (VSS), U5.16 (VCC), U6.16 (VCC), U68.20 (VCC), U69.20 (VCC), U70.20 (VCC), U71.20 (VCC), U82.7 (VCC), U83.20 (VCC), U84.20 (VCC), U89.14 (VCC), U90.14 (VCC), U97.20 (VCC), U98.20 (VCC), U99.16 (VCC)
- net CCLK: now also U23.11 (Q3), U39.3
- net D0: now also U69.11, U82.31 (D0)
- net D2: now also U69.13, U82.29 (D2)
- net D3: now also U69.14, U82.28 (D3)
- net D5: now also U69.16, U82.26 (D5)
- net D6: now also U69.17, U82.25 (D6)
- net D7: now also U69.18, U82.24 (D7)
- net DA0: now also U21.6
- net DA1: now also U21.3
- net DA2: now also U6.13
- net DA3: now also U6.10
- net DA4: now also U6.6
- net DA5: now also U6.3
- net DA6: now also U5.13
- net DA7: now also U5.10
- net DA8: now also U5.6
- net DA9: now also U5.3
- net DD0: now also U2.11
- net DD1: now also U2.12
- net DD2: now also U2.13
- net DD3: now also U2.14
- net DD4: now also U2.15
- net DD5: now also U2.16
- net DD6: now also U2.17
- net DD7: now also U2.18
- net DRW: now also U2.1 (D), U21.13
- net E: now also U25.6, U37.4
- net GND: now also C14.2, C31.2, R2.2, R37.2, SW1.2, U1.10 (GND), U101.10, U101.9, U2.10 (GND), U21.15 (~E), U21.8 (GND), U22.7 (GND), U23.3, U23.4, U23.5, U23.6, U23.8 (GND), U24.7 (GND), U25.1 (~OE), U25.10 (GND), U3.9 (GND), U36.7 (GND), U37.7 (GND), U38.7 (GND), U39.5, U39.7 (GND), U4.9 (GND), U5.15 (~E), U5.8 (GND), U6.15 (~E), U6.8 (GND), U68.1 (~E1), U68.10 (GND), U68.19 (~E2), U69.10 (GND), U70.10 (GND), U71.10 (GND), U82.1 (GND), U82.39 (TSC), U83.1 (~E1), U83.10 (GND), U83.19 (~E2), U84.10 (GND), U88.12, U88.13, U89.3 (1CLK), U89.7 (GND), U9.12, U9.13, U90.1, U90.13, U90.3, U90.7 (GND), U97.1 (~E1), U97.10 (GND), U97.19 (~E2), U98.10 (GND), U99.8 (GND)
- net LA10: now also U70.15, U98.16
- net LA11: now also U70.12, U98.5
- net LA12: now also U70.9, U98.12
- net LA13: now also U70.6, U98.9
- net LA14: now also U70.5, U98.7
- net LA15: now also U36.5 (1Q)
- net LA2: now also U71.15, U84.7
- net LA3: now also U71.12, U84.14
- net LA4: now also U71.9, U84.5
- net LA5: now also U71.6, U84.16
- net LA6: now also U71.5, U84.3
- net LA7: now also U71.2, U84.18
- net LA8: now also U70.19, U98.18
- net LA9: now also U70.16, U98.3
- net Q: now also U25.2, U25.4, U37.1, U9.9
- net QX: now also U24.9, U25.5, U25.7, U9.10
- net RP6: now also U23.1, U23.10, U23.7, U23.9, U36.1 (~1CLR), U36.4 (~1PRE_), U38.10 (S), U38.2 (K), U38.3 (J), U38.4 (S)
- net VA0: now also U21.5, U83.9, U84.11
- net VA1: now also U21.2, U83.12, U84.8
- net VA10: now also U97.16, U98.4, U99.1 (A0)
- net VA11: now also U97.5, U98.15, U99.2 (A1)
- net VA12: now also U97.12, U98.8, U99.3 (A2)
- net VA13: now also U97.9, U98.11, U99.4 (E1)
- net VA14: now also U97.7, U98.13, U99.5 (E2)
- net VA15: now also TP8.1, U97.14, U98.6, U99.6 (E3)
- net VA2: now also U6.14, U83.7, U84.13
- net VA3: now also U6.11, U83.14, U84.6
- net VA4: now also U6.5, U83.5, U84.15
- net VA5: now also U6.2, U83.16, U84.4
- net VA6: now also U5.14, U83.3, U84.17
- net VA7: now also U5.11, U83.18, U84.2
- net VA8: now also U5.5, U97.18, U98.2
- net VA9: now also U5.2, U97.3, U98.17
- net VBA: now also U68.14
- net VBS: now also U68.5
- net VBSC: now also R67.2, TP7.1, U90.11
- net VD0: now also U1.11, U69.9, U70.18, U71.18
- net VD1: now also U1.12, U69.8, U70.17, U71.17
- net VD2: now also U1.13, U69.7, U70.14, U71.14
- net VD3: now also U1.14, U69.6, U70.13, U71.13
- net VD4: now also U1.15, U69.5, U70.8, U71.8
- net VD5: now also U1.16, U69.4, U70.7, U71.7
- net VD6: now also U1.17, U69.3, U70.4, U71.4
- net VD7: now also U1.18, U36.2 (1D), U69.2, U71.3
- net VE: now also R63.1, TP4.1, U37.6, U82.34 (E)
- net VLIC: now also U68.16
- net VMA: now also U68.3
- net VQ: now also TP3.1, U37.3, U82.35 (Q)
- net VRW: now also U1.1 (D), U22.1, U22.4, U68.7, U69.1 (D)
- net ~CAS: now also U25.19
- net ~CCLK: now also U39.4
- net ~MRST: now also R37.1, U68.2, U82.37 (~RST)
- net ~MUX: now also U37.9, U38.8 (~Q)
- net ~QRW: now also U22.6
- net ~QX: now also U24.8, U25.13
- net ~RAS: now also U37.8
- net ~VFIRQ: now also U82.4 (~FIRQ)
- net ~VHALT: now also R60.2, U82.40 (~HALT)
- net ~VIRQ: now also SW1.1, U82.3 (~IRQ)
- net ~VNMI: now also U82.2 (~NMI)
- net ~VRST: now also U68.18
- net ~VS2: now also U99.13
- net ~VS6: now also U99.9
- net ~VS7: now also U99.7
- new net: TP6.1, U82.33 (BUSY)
- new net: R59.1, U69.12, U82.30 (D1)
- new net: R50.2, U69.15, U82.27 (D4)
- new net: U69.19 (~E), U90.10
- new net: U82.21 (A13), U97.11
- new net: U82.22 (A14), U97.13
- new net: U82.19 (A11), U97.15
- new net: U82.17 (A9), U97.17
- new net: U82.16 (A8), U97.2
- new net: U82.18 (A10), U97.4
- new net: U82.23 (A15), U97.6
- new net: U82.20 (A12), U97.8
- new net: U82.8 (A0), U83.11
- new net: U82.10 (A2), U83.13
- new net: U82.12 (A4), U83.15
- new net: U82.14 (A6), U83.17
- new net: U82.15 (A7), U83.2
- new net: U82.13 (A5), U83.4
- new net: U82.11 (A3), U83.6
- new net: U82.9 (A1), U83.8
- new net: U68.13, U82.32 (R/~W)
- new net: U68.15, U82.5 (BS)
- new net: U68.17, U82.36 (AVMA)
- new net: TP5.1, U68.4, U82.38 (LIC)
- new net: U68.6, U82.6 (BA)
- new net: C31.1, R2.1, R8.2, U24.1, Y1.1
- new net: C14.1, Y1.2
- new net: R7.2, R8.1, U24.2, U39.1
- new net: U38.1 (C), U39.2
- new net: TP2.1, U23.2 (C), U25.11 (C), U38.13 (C), U38.5 (Q)
- new net: U23.12 (Q2), U24.11, U25.3
- new net: U23.13 (Q1), U24.5, U37.13
- new net: U23.14 (Q0), U24.3, U38.11 (J)
- new net: U24.10, U25.14
- new net: U24.6, U25.8
- new net: U25.17, U9.8
- new net: U25.18, U37.11
- new net: U25.9, U37.10, U37.12, U38.12 (K)
- new net: U1.19 (~E), U22.11
- new net: U1.2, U2.2, U3.11 (D4)
- new net: U1.3, U2.3, U3.12 (D3)
- new net: U1.4, U2.4, U3.13 (D2)
- new net: U1.5, U2.5, U3.14 (D1)
- new net: U1.6, U2.6, U4.11 (D4)
- new net: U1.7, U2.7, U4.12 (D3)
- new net: U1.8, U2.8, U4.13 (D2)
- new net: U1.9, U2.9, U4.14 (D1)
- new net: U3.1 (A6), U4.1 (A6), U5.12
- new net: U22.8, U3.10 (WE_), U4.10 (WE_)
- new net: U3.15 (A9), U4.15 (A9), U5.4
- new net: U3.16 (A8), U4.16 (A8), U5.7
- new net: U3.17 (A7), U4.17 (A7), U5.9
- new net: U3.2 (A5), U4.2 (A5), U6.4
- new net: U3.3 (A4), U4.3 (A4), U6.7
- new net: U3.4 (A3), U4.4 (A3), U6.9
- new net: U21.7, U3.5 (A0), U4.5 (A0)
- new net: U21.4, U3.6 (A1), U4.6 (A1)
- new net: U3.7 (A2), U4.7 (A2), U6.12
- new net: U21.9, U22.9, U4.8 (CS)
- new net: U21.12, U22.10
- new net: U21.14, U22.3
- new net AEN: U70.1 (~OE), U71.1 (~OE)
- new net DPMUX: U2.19 (~E), U36.9 (2Q), U37.2, U37.5
- new net LA0: U71.19, U84.9
- new net LA1: U71.16, U84.12
- new net MUX: U36.11 (2CLK), U38.9 (Q)
- new net PR6: U36.10 (~1PRE_), U36.13 (~1CLR)
- new net PR62: U89.1 (~1CLR), U89.4 (~1PRE_)
- new net VBQ: U25.16
- new net ~5MHZ: U24.4
- new net ~AEN: U84.1 (~E1), U84.19 (~E2), U98.1 (~E1), U98.19 (~E2)
- new net ~ASH: U36.3 (1CLK), U70.11 (C)
- new net ~ASL: U71.11 (C)
- new net ~DPMUX: U21.1 (S), U22.13, U36.8 (~2Q), U5.1 (S), U6.1 (S)
- new net ~DS0: U36.12 (2D)
- new net ~E: U21.11, U25.12
- new net ~Q: U21.10, U22.5, U25.15
- new net ~VS0: U22.12, U22.2, U99.15
- new net ~VS1: U99.14
- new net ~VS3: U99.12
- new net ~VS4: U99.11
- new net ~VS5: U99.10
- no-connect marks 37 -> 57
Other:
- moved on the sheet: C22, C42, C44, C45, C9, J6, R1, R10, R51, R52, R53, R54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

Commit message: Fixed several schematic errors
Parts:
- added unit 5 of U39
- added unit 6 of U39
- added U7: LS74, symbol Asteroids:LS74
- added U8: LS32, symbol Asteroids:LS32
- added unit 2 of U9
- added unit 1 of U9
Connections:
- net RP6 is gone; now on net PR6: R6.2, U23.1, U23.10, U23.7, U23.9, U36.1 (~1CLR), U36.4 (~1PRE_), U38.10 (S), U38.2 (K), U38.3 (J), U38.4 (S)
- net RP62 is gone; now on net PR62: R62.2
- net vEQ is gone; now on net VEQ: U101.4
- net +5V: now also U7.14 (VCC), U8.14 (VCC), U9.14 (VCC)
- net DA0: now also U39.13, U8.1
- net GND: now also U7.12 (2D), U7.2 (1D), U7.7 (GND), U8.7 (GND), U9.7 (GND)
- net VA0: now also U39.11, U8.9
- net ~DS3: now also U9.1
- net ~E: now also U9.4
- net ~Q: now also U9.2
- net ~VFIRQ: now also U7.8 (~2Q)
- net ~VRST: now also U7.1 (~1CLR), U7.13 (~1CLR)
- net ~VS3: now also U9.5
- net RP68 renamed PR68
- net RP69 renamed PR69
- new net: U8.13, U8.2, U9.3
- new net: U7.10 (~1PRE_), U8.3
- new net: U39.10, U8.4
- new net: U8.10, U8.5, U9.6
- new net: U7.11 (2CLK), U8.6
- new net: U7.4 (~1PRE_), U8.8
- new net: U7.3 (1CLK), U8.11
- new net: U39.12, U8.12
- new net ~DFIRQ: U7.6 (~1Q)
- no-connect marks 57 -> 59
Other:
- moved on the sheet: C14, C31, R2, R7, R8, TP2, U23, U24A, U24B, U24C, U24D, U24E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

Commit message: Completed schematic capture - still need to fix ERC errors
Parts:
- added C113, C96, C97, C98: 470pf, symbol Device:C
- added C61, C63, C77, C80: 10uf, symbol Device:CP1
- added C88, C89, C90: 100uf, symbol Device:CP1
- added FB1, FB10, FB14, FB2, FB3, FB4, FB5, FB6, FB8, FB9: Ferrite_Bead, symbol Device:Ferrite_Bead
- added J1, J2: 14pin, symbol taito_pcb:14pin
- added Q1, Q2, Q3, Q4, Q5, Q6, Q7: 2N3904, Package_TO_SOT_THT:TO-92_Inline, symbol Transistor_BJT:2N3904
- added R13, R20, R46: 82, symbol Device:R_US
- added R14, R19, R28, R48: 180, symbol Device:R_US
- added R15, R18, R3, R4, R49, R5: 270, symbol Device:R_US
- added R16, R17, R45: 150, symbol Device:R_US
- added R21, R36: 33, symbol Device:R_US
- added R29, R30, R31, R32, R33, R47: 470, symbol Device:R_US
- added R34: 680, symbol Device:R_US
- added R35: 390, symbol Device:R_US
- added TP1: TestPoint, symbol Connector:TestPoint
- added unit 4 of U101
- added unit 3 of U102
- added unit 2 of U102
- added unit 2 of U103
- added unit 3 of U103
- added unit 4 of U103
- added U104, U55, U73, U74, U81: 157_1, symbol taito_pcb:157_1
- added U105, U106, U107, U108, U109, U110, U95, U96: 299_1, symbol taito_pcb:299_1
- added unit 6 of U24
- added unit 5 of U40
- added unit 4 of U40
- added unit 1 of U40
- added unit 3 of U40
- added unit 2 of U40
- added U41, U42, U43, U44, U45, U46, U47, U48, U59, U60, U61, U62, U63, U64, U65, U66: 4116, symbol taito_pcb:4116
- added unit 4 of U51
- added U56: 2148_1, symbol taito_pcb:2148_1
- added U57: 2148_2, symbol taito_pcb:2148_2
- added U58: 7417, symbol taito_pcb:7417
- added U67: LS32, symbol Asteroids:LS32
- added U75: 245_1, symbol taito_pcb:245_1
- added U76: 273_1, symbol taito_pcb:273_1
- added U79, U80: 373, symbol taito_pcb:373
- added U87: LS139, symbol Asteroids:LS139
- added unit 3 of U88
- added unit 2 of U88
- added unit 2 of U89
- added unit 3 of U90
- added unit 4 of U90
- added U91, U92, U93, U94: 374_1, symbol taito_pcb:374_1
Connections:
- net VBQ is gone; now on net VEQ: U25.16
- net ~DEIRQ is gone; now on net ~DFIRQ: J6.43
- net ~DS1 is gone; now on net ~DS0: J6.27
- net +12V: now also C61.1, C77.1, C89.1, FB10.2, U41.8, U42.8, U43.8, U44.8, U45.8, U46.8, U47.8, U48.8, U59.8, U60.8, U61.8, U62.8, U63.8, U64.8, U65.8, U66.8
- net +5V: now also U34.20 (VCC), C90.1, FB8.2, Q1.3 (C), R28.2, R3.1, R4.1, R5.1, U104.16 (VCC), U105.20 (VCC), U106.20 (VCC), U107.20 (VCC), U108.20 (VCC), U109.20 (VCC), U110.20 (VCC), U40.14 (VCC), U41.9, U42.9, U43.9, U44.9, U45.9, U46.9, U47.9, U48.9, U55.16 (VCC), U56.18 (VCC), U57.18 (VCC), U58.14 (VCC), U59.9, U60.9, U61.9, U62.9, U63.9, U64.9, U65.9, U66.9, U67.14 (VCC), U73.16 (VCC), U74.16 (VCC), U75.20 (VCC), U76.20 (VCC), U79.20 (VCC), U80.20 (VCC), U81.16 (VCC), U87.16 (VCC), U91.20 (VCC), U92.20 (VCC), U93.20 (VCC), U94.20 (VCC), U95.20 (VCC), U96.20 (VCC)
- net -5V: now also C63.2, C80.2, C88.2, FB9.2, U41.1, U42.1, U43.1, U44.1, U45.1, U46.1, U47.1, U48.1, U59.1, U60.1, U61.1, U62.1, U63.1, U64.1, U65.1, U66.1
- net AEN: now also U101.13, U88.6, U90.9
- net BD0: now also U48.2, U66.2
- net BD1: now also U47.2, U65.2
- net BD2: now also U46.2, U64.2
- net BD3: now also U45.2, U63.2
- net BD4: now also U44.2, U62.2
- net BD5: now also U43.2, U61.2
- net BD6: now also U42.2, U60.2
- net BD7: now also U41.2, U59.2
- net CCLK: now also U102.3
- net CR8: now also U55.6
- net CR9: now also U55.3
- net E: now also U102.9, U103.12, U91.11 (C), U92.11 (C), U93.11 (C), U94.11 (C)
- net GND: now also U34.10 (GND), C113.2, C61.2, C63.1, C77.2, C80.1, C88.1, C89.2, C90.2, C96.2, C97.2, C98.2, J1.11, J1.3, J1.5, J1.7, J2.4, R16.1, R17.1, R45.1, U104.15 (~E), U104.8 (GND), U105.10 (GND), U106.10 (GND), U107.10 (GND), U108.10 (GND), U109.10 (GND), U110.10 (GND), U40.7 (GND), U41.16, U42.16, U43.16, U44.16, U45.16, U46.16, U47.16, U48.16, U55.15 (~E), U55.8 (GND), U56.8 (~CE), U56.9 (GND), U57.8 (~CE), U57.9 (GND), U58.7 (GND), U59.16, U60.16, U61.16, U62.16, U63.16, U64.16, U65.16, U66.16, U67.7 (GND), U73.15 (~E), U73.8 (GND), U74.10, U74.15 (~E), U74.8 (GND), U75.10 (GND), U76.10 (GND), U79.10 (GND), U80.10 (GND), U81.15 (~E), U81.8 (GND), U87.8 (GND), U91.1 (~OE), U91.10 (GND), U92.1 (~OE), U92.10 (GND), U93.1 (~OE), U93.10 (GND), U94.1 (~OE), U94.10 (GND), U95.10 (GND), U96.10 (GND)
- net HS: now also U40.1
- net INV: now also TP1.1, U103.9, U104.1 (S), U24.13, U81.1 (S)
- net LA0: now also U87.14 (2A)
- net LA1: now also U87.13 (2B)
- net M0: now also U41.5, U42.5, U43.5, U44.5, U45.5, U46.5, U47.5, U48.5, U59.5, U60.5, U61.5, U62.5, U63.5, U64.5, U65.5, U66.5
- net M1: now also U41.6, U42.6, U43.6, U44.6, U45.6, U46.6, U47.6, U48.6, U59.6, U60.6, U61.6, U62.6, U63.6, U64.6, U65.6, U66.6
- net M2: now also U41.7, U42.7, U43.7, U44.7, U45.7, U46.7, U47.7, U48.7, U59.7, U60.7, U61.7, U62.7, U63.7, U64.7, U65.7, U66.7
- net M3: now also U41.12, U42.12, U43.12, U44.12, U45.12, U46.12, U47.12, U48.12, U59.12, U60.12, U61.12, U62.12, U63.12, U64.12, U65.12, U66.12
- net M4: now also U41.11, U42.11, U43.11, U44.11, U45.11, U46.11, U47.11, U48.11, U59.11, U60.11, U61.11, U62.11, U63.11, U64.11, U65.11, U66.11
- net M5: now also U41.10, U42.10, U43.10, U44.10, U45.10, U46.10, U47.10, U48.10, U59.10, U60.10, U61.10, U62.10, U63.10, U64.10, U65.10, U66.10
- net M6: now also U41.13, U42.13, U43.13, U44.13, U45.13, U46.13, U47.13, U48.13, U59.13, U60.13, U61.13, U62.13, U63.13, U64.13, U65.13, U66.13
- net PR62: now also U89.10 (~1PRE_), U89.13 (~1CLR)
- net PR68: now also U105.9, U106.9, U107.9, U108.9, U109.9, U110.9, U95.9, U96.9
- net PR69: now also U105.2, U105.3, U106.2, U106.3, U107.2, U107.3, U108.2, U108.3, U109.2, U109.3, U110.2, U110.3, U95.2, U95.3, U96.2, U96.3
- net Q: now also U102.5
- net QX: now also U79.11 (C), U80.11 (C)
- net R0: now also U108.7, U92.18
- net R1: now also U107.7, U92.17
- net R10: now also U106.13, U91.14
- net R11: now also U105.13, U91.13
- net R12: now also U91.8, U96.13
- net R13: now also U91.7, U95.13
- net R14: now also U110.13, U91.4
- net R15: now also U109.13, U91.3
- net R2: now also U106.7, U92.14
- net R3: now also U105.7, U92.13
- net R4: now also U92.8, U96.7
- net R5: now also U92.7, U95.7
- net R6: now also U110.7, U92.4
- net R7: now also U109.7, U92.3
- net R8: now also U108.13, U91.18
- net R9: now also U107.13, U91.17
- net VA0: now also U74.5, U87.2 (1A)
- net VA1: now also U74.2, U87.3 (1B), U88.4
- net VA15: now also U101.12
- net VA2: now also U73.14
- net VA3: now also U73.11
- net VA4: now also U73.5
- net VA5: now also U73.2
- net VA6: now also U55.14
- net VA7: now also U55.11
- net VA8: now also U55.5
- net VA9: now also U55.2
- net VD0: now also U75.11, U79.19, U80.19
- net VD1: now also U75.12, U79.16, U80.16
- net VD2: now also U75.13, U79.15, U80.15
- net VD3: now also U75.14, U79.12, U80.12
- net VD4: now also U75.15, U79.9, U80.9
- net VD5: now also U75.16, U79.6, U80.6
- net VD6: now also U75.17, U79.5, U80.5
- net VD7: now also U75.18, U79.2, U80.2
- net VEN: now also U89.12 (2D)
- net VRW: now also U90.5
- net VS: now also U40.5
- net _VS: now also FB1.2, R3.2, R5.2, U40.6, U51.13
- net ~5MHZ: now also U105.12 (CLK), U106.12 (CLK), U107.12 (CLK), U108.12 (CLK), U109.12 (CLK), U110.12 (CLK), U76.11 (C), U95.12 (CLK), U96.12 (CLK)
- net ~AEN: now also U90.8
- net ~ASH: now also U87.6 (1Y2)
- net ~ASL: now also U87.7 (1Y3)
- net ~CAS: now also U41.15, U42.15, U43.15, U44.15, U45.15, U46.15, U47.15, U48.15, U59.15, U60.15, U61.15, U62.15, U63.15, U64.15, U65.15, U66.15
- net ~E: now also U102.4
- net ~EVEN0: now also U87.12 (2Y0)
- net ~INV: now also U103.4, U24.12
- net ~MRST: now also FB14.2
- net ~ODD0: now also U87.11 (2Y1)
- net ~QRW: now also U88.9
- net ~RAS: now also U41.4, U42.4, U43.4, U44.4, U45.4, U46.4, U47.4, U48.4, U59.4, U60.4, U61.4, U62.4, U63.4, U64.4, U65.4, U66.4
- net ~VEW: now also U103.11, U67.1, U67.4
- net ~VRW: now also U103.13, U67.12, U67.9, U74.11, U90.6
- net ~VS4: now also U55.1 (S), U73.1 (S), U74.1 (S), U75.19 (~E)
- net ~VS5: now also U88.10, U88.5
- net at C14.1, Y1.2: now also R7.1
- new net: U55.12, U56.1, U57.1
- new net: U55.4, U56.15, U57.15
- new net: U55.7, U56.16, U57.16
- new net: U55.9, U56.17, U57.17
- new net: U56.7, U57.7, U73.12
- new net: U56.2, U57.2, U73.4
- new net: U56.3, U57.3, U73.7
- new net: U56.4, U57.4, U73.9
- new net: U56.6, U57.6, U74.4
- new net: U56.5, U57.5, U74.7
- new net: U102.10, U102.11, U74.9
- new net: U102.8, U56.10 (RW), U75.1 (D)
- new net: U56.11, U75.2, U76.18
- new net: U56.12, U75.3, U76.17
- new net: U56.13, U75.4, U76.14
- new net: U56.14, U75.5, U76.13
- new net: U57.12, U75.6, U76.8
- new net: U57.13, U75.7, U76.7
- new net: U57.11, U75.8, U76.4
- new net: U57.14, U75.9, U76.3
- new net: U76.1 (~R), U89.9 (2Q)
- new net: Q1.1 (E), Q2.3 (C), Q3.3 (C), R29.1, R30.1
- new net: Q1.2 (B), R28.1, R34.2, R35.2
- new net: Q2.1 (E), R14.1
- new net: Q2.2 (B), R29.2, U58.2
- new net: Q4.1 (E), R19.1
- new net: Q4.2 (B), R32.2, U40.8
- new net: Q4.3 (C), Q5.3 (C), R31.1, R32.1
- new net: Q6.1 (E), R48.1
- new net: Q6.2 (B), R33.2, U58.10
- new net: Q6.3 (C), Q7.3 (C), R33.1, R47.1
- new net: Q3.1 (E), R13.1
- new net: Q3.2 (B), R30.2, U40.10
- new net: Q5.1 (E), R20.1
- new net: Q5.2 (B), R31.2, U58.12
- new net: Q7.1 (E), R46.1
- new net: Q7.2 (B), R47.2, U58.8
- new net: R34.1, U58.6
- new net: R35.1, U58.4
- new net: U58.5, U76.2
- new net: U58.3, U76.5
- new net: U58.1, U76.6
- new net: U40.11, U76.9
- new net: U40.9, U76.12
- new net: U58.13, U76.15
- new net: U58.11, U76.16
- new net: U58.9, U76.19
- new net: R13.2, R14.2, R15.2, R16.2
- new net: FB4.2, R15.1
- new net: R17.2, R18.2, R19.2, R20.2
- new net: FB5.2, R18.1
- new net: R45.2, R46.2, R48.2, R49.2
- new net: FB6.2, R49.1
- new net: R21.1, U41.3, U42.3, U43.3, U44.3, U45.3, U46.3, U47.3, U48.3
- new net: U67.8, U79.1 (~OE)
- new net: R21.2, U67.6
- new net: R36.1, U59.3, U60.3, U61.3, U62.3, U63.3, U64.3, U65.3, U66.3
- new net: U67.11, U80.1 (~OE)
- new net: R36.2, U67.3
- new net: U87.1 (1G), U88.8
- new net: U101.11, U87.15 (2G)
- new net: FB3.2, U40.2, U51.12
- new net: U40.3, U51.11
- new net: FB2.2, R4.2, U40.4
- new net CR0: U104.12, U74.6
- new net CR1: U104.9, U74.3
- new net CR2: U104.7, U73.13
- new net CR3: U104.4, U73.10
- new net CR4: U73.6, U81.12
- new net CR5: U73.3, U81.9
- new net CR6: U55.13, U81.7
- new net CR7: U55.10, U81.4
- new net LS: U102.6, U103.10, U103.5, U89.11 (2CLK)
- new net R16: U108.6, U66.14, U80.18, U94.18
- new net R17: U107.6, U65.14, U80.17, U94.17
- new net R18: U106.6, U64.14, U80.14, U94.14
- new net R19: U105.6, U63.14, U80.13, U94.13
- new net R20: U62.14, U80.8, U94.8, U96.6
- new net R21: U61.14, U80.7, U94.7, U95.6
- new net R22: U110.6, U60.14, U80.4, U94.4
- new net R23: U109.6, U59.14, U80.3, U94.3
- new net R24: U108.14, U48.14, U79.18, U93.18
- new net R25: U107.14, U47.14, U79.17, U93.17
- new net R26: U106.14, U46.14, U79.14, U93.14
- new net R27: U105.14, U45.14, U79.13, U93.13
- new net R28: U44.14, U79.8, U93.8, U96.14
- new net R29: U43.14, U79.7, U93.7, U95.14
- new net R30: U110.14, U42.14, U79.4, U93.4
- new net R31: U109.14, U41.14, U79.3, U93.3
- new net R32: U108.5, U92.19
- new net R33: U107.5, U92.16
- new net R34: U106.5, U92.15
- new net R35: U105.5, U92.12
- new net R36: U92.9, U96.5
- new net R37: U92.6, U95.5
- new net R38: U110.5, U92.5
- new net R39: U109.5, U92.2
- new net R40: U108.15, U91.19
- new net R41: U107.15, U91.16
- new net R42: U106.15, U91.15
- new net R43: U105.15, U91.12
- new net R44: U91.9, U96.15
- new net R45: U91.6, U95.15
- new net R46: U110.15, U91.5
- new net R47: U109.15, U91.2
- new net R48: U108.4, U94.19
- new net R49: U107.4, U94.16
- new net R50: U106.4, U94.15
- new net R51: U105.4, U94.12
- new net R52: U94.9, U96.4
- new net R53: U94.6, U95.4
- new net R54: U110.4, U94.5
- new net R55: U109.4, U94.2
- new net R56: U108.16, U93.19
- new net R57: U107.16, U93.16
- new net R58: U106.16, U93.15
- new net R59: U105.16, U93.12
- new net R60: U93.9, U96.16
- new net R61: U93.6, U95.16
- new net R62: U110.16, U93.5
- new net R63: U109.16, U93.2
- new net S0: U103.6, U105.1 (S0), U106.1 (S0), U107.1 (S0), U108.1 (S0), U109.1 (S0), U110.1 (S0), U95.1 (S0), U96.1 (S0)
- new net S1: U103.8, U105.19 (S1), U106.19 (S1), U107.19 (S1), U108.19 (S1), U109.19 (S1), U110.19 (S1), U95.19 (S1), U96.19 (S1)
- new net _+12V_: C98.1, FB10.1, J1.6
- new net _+5V_: C96.1, FB8.1, J1.1, J1.2
- new net _-5V_: C97.1, FB9.1, J1.4
- new net _00: U104.13, U108.17
- new net _01: U104.14, U108.8
- new net _02: U104.10, U107.17
- new net _03: U104.11, U107.8
- new net _04: U104.6, U106.17
- new net _05: U104.5, U106.8
- new net _06: U104.3, U105.17
- new net _07: U104.2, U105.8
- new net _10: U81.13, U96.17
- new net _11: U81.14, U96.8
- new net _12: U81.10, U95.17
- new net _13: U81.11, U95.8
- new net _14: U110.17, U81.6
- new net _15: U110.8, U81.5
- new net _16: U109.17, U81.3
- new net _17: U109.8, U81.2
- new net _BLUE_: FB4.1, J2.10
- new net _CS_: FB2.1, J2.2
- new net _GREEN_: FB5.1, J2.11
- new net _HS_: FB3.1, J2.9
- new net _MRST_: C113.1, FB14.1, J1.14
- new net _RED_: FB6.1, J2.14
- new net _VS_: FB1.1, J2.1
- new net ~EVEN1: U67.13, U67.2, U87.10 (2Y2)
- new net ~ODD1: U67.10, U67.5, U87.9 (2Y3)
- no-connect marks 59 -> 93
Other:
- moved on the sheet: C22, C42, C44, C45, C9, R1, R10, R51, R52, R53, R54, R55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

Commit message: Began PCB layout and added all ICs
Parts:
- Q1, Q2, Q3, Q4, Q5, Q6, Q7: footprint Package_TO_SOT_THT:TO-92_Inline -> (none)
- U1, U105, U106, U107, U108, U109, U110, U2, U25, U34, U68, U69, U70, U71, U72, U75, U76, U77, U78, U79, U80, U83, U84, U91, U92, U93, U94, U95, U96, U97, U98: footprint (none) -> Star_Wars_Vector_PCB:DIP20
- U10, U104, U11, U12, U13, U14, U15, U16, U17, U21, U23, U26, U27, U28, U29, U30, U31, U32, U33, U35, U41, U42, U43, U44, U45, U46, U47, U48, U5, U52, U53, U54, U55, U59, U6, U60, U61, U62, U63, U64, U65, U66, U73, U74, U81, U87, U99: footprint (none) -> Star_Wars_Vector_PCB:DIP16
- U100, U101, U102, U103, U19, U20, U22, U24, U36, U37, U38, U39, U40, U49, U50, U51, U58, U67, U7, U8, U88, U89, U9, U90: footprint (none) -> Star_Wars_Vector_PCB:DIP14
- U18, U82: footprint (none) -> Star_Wars_Vector_PCB:DDIP40
- U3, U4, U56, U57, U85, U86: footprint (none) -> Star_Wars_Vector_PCB:DIP18
Connections:
- net ~VSI is gone; now on net ~VS1: U39.9
- net at U102.8, U56.10 (RW), U75.1 (D): now also U57.10 (RW)
- net at U3.8 (CS): now also U21.9, U22.9, U4.8 (CS)
Other:
- moved on the sheet: BT1, C101, C113, C14, C22, C31, C42, C44, C45, C61, C63, C65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
