File: taito_video_processor_pcb/taito_video_processor_pcb.kicad_pcb (KiCad board)
At the start: 2 copper layers, 304.8 x 279.4 mm, 352 parts, among them J1 14pin, J19 2pin, J2 14pin, J3 50pin, J6 50pin, Q1 2N3904, Q2 2N3904, Q3 2N3904, Q4 2N3904, Q5 2N3904, Q6 2N3904, Q7 2N3904, Q8 2N3905, SW1 SW_Push, U1 245_1, U10 4116, U100 LS00, U101 LS08, U102 LS10, U103 LS00, U104 157_1, U105 299_1, U106 299_1, U107 299_1, U108 299_1, U109 299_1, U11 4116, U110 299_1, U12 4116, U13 4116, U14 4116, U15 4116, U16 4116, U17 4116, U18 68A45, U19 86_2, U2 245_1, U20 86_1, U21 157_1, U22 LS32, U23 161_1, U24 LS04, U25 374_1, U26 4116, U27 4116, U28 4116, U29 4116, U3 2114, U30 4116, U31 4116, U32 4116, U33 4116, U34 LS374, U35 153_1, U36 LS74, U37 LS08, U38 74S113, U39 LS04, U4 2114, U40 7417, U41 4116, U42 4116, U43 4116, U44 4116, U45 4116, U46 4116, U47 4116, U48 4116, U49 LS32, U5 157_1, U50 86_3, U51 LS86, U52 153_1, U53 153_1, U54 153_1, U55 157_1, U56 2148_1, U57 2148_2, U58 7417, U59 4116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

Commit message: Added more traces
Parts:
- moved C81 1.91 mm to (413.4, 193.0)
- moved C80 1.27 mm to (408.3, 198.8)
- moved C53 0.64 mm to (307.3, 163.2)
- moved C62 0.64 mm to (398.8, 163.2)
- moved C54 0.63 mm to (321.3, 161.9)
- moved C57 0.63 mm to (336.6, 162.6)
- moved C58 0.63 mm to (351.8, 162.6)
- turned C64 to 180 degrees
Connections:
- C41 pad 1: +5V -> +12V
- R5 pad 2: _VS -> Net-(FB3-Pad2)
- R9 pad 1: ~CAS1 -> ~CAS
- R9 pad 2: ~CAS -> Net-(R9-Pad2)
- RP1 pad 2: ~CAS1 -> ~CAS
- U25 pad 19: ~CAS -> Net-(R9-Pad2)
Routing:
- net GND: track 341.4 -> 820.0 mm, vias 18 -> 19
- net M3: track 0.00 -> 361.8 mm
- net M6: track 0.00 -> 357.3 mm, vias 0 -> 1
- net M5: track 0.00 -> 356.1 mm
- net M4: track 0.00 -> 354.7 mm
- net M2: track 0.00 -> 347.0 mm
- net M1: track 0.00 -> 345.9 mm
- net M0: track 0.00 -> 345.9 mm
- net +5V: track 370.0 -> 705.7 mm
- net +12V: track 140.0 -> 419.0 mm, vias 7 -> 17
- net ~CAS: track 0.00 -> 268.3 mm
- net ~RAS: track 0.00 -> 235.1 mm
- net -5V: track 224.0 -> 452.0 mm
- net Net-(FB2-Pad2): track 0.00 -> 142.1 mm
- net _VS: track 0.00 -> 137.6 mm
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