File: taito_video_processor_pcb/taito_video_processor_pcb.kicad_pcb (KiCad board)
At the start: 2 copper layers, 304.8 x 279.4 mm, 352 parts, among them J1 14pin, J19 2pin, J2 14pin, J3 50pin, J6 50pin, Q1 2N3904, Q2 2N3904, Q3 2N3904, Q4 2N3904, Q5 2N3904, Q6 2N3904, Q7 2N3904, Q8 2N3905, SW1 SW_Push, U1 245_1, U10 4116, U100 LS00, U101 LS08, U102 LS10, U103 LS00, U104 157_1, U105 299_1, U106 299_1, U107 299_1, U108 299_1, U109 299_1, U11 4116, U110 299_1, U12 4116, U13 4116, U14 4116, U15 4116, U16 4116, U17 4116, U18 68A45, U19 86_2, U2 245_1, U20 86_1, U21 157_1, U22 LS32, U23 161_1, U24 LS04, U25 374_1, U26 4116, U27 4116, U28 4116, U29 4116, U3 2114, U30 4116, U31 4116, U32 4116, U33 4116, U34 LS374, U35 153_1, U36 LS74, U37 LS08, U38 74S113, U39 LS04, U4 2114, U40 7417, U41 4116, U42 4116, U43 4116, U44 4116, U45 4116, U46 4116, U47 4116, U48 4116, U49 LS32, U5 157_1, U50 86_3, U51 LS86, U52 153_1, U53 153_1, U54 153_1, U55 157_1, U56 2148_1, U57 2148_2, U58 7417, U59 4116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

Commit message: 1285 signal left to connect
Parts:
- moved R49 0.64 mm to (307.3, 231.1)
- moved C73 0.63 mm to (322.6, 198.8)
- moved C74 0.63 mm to (337.8, 198.8)
- moved C78 0.63 mm to (398.8, 198.8)
- moved C80 0.63 mm to (408.3, 198.1)
- moved U93 0.13 mm to (353.1, 287.0)
- moved U94 0.13 mm to (368.3, 287.0)
- moved U95 0.13 mm to (383.5, 287.0)
Connections:
- U67 pad 2: ~ODD1 -> ~EVEN1
- U67 pad 3: Net-(R21-Pad2) -> Net-(R36-Pad2)
- U67 pad 5: ~EVEN1 -> ~ODD1
- U67 pad 6: Net-(R36-Pad2) -> Net-(R21-Pad2)
Routing:
- net GND: track 820.0 -> 1931.9 mm
- net +5V: track 705.7 -> 1464.4 mm, vias 0 -> 1
- net +12V: track 419.0 -> 558.6 mm
- net Net-(R36-Pad1): track 0.00 -> 127.8 mm
- net M6: track 357.3 -> 471.4 mm
- net M4: track 354.7 -> 468.8 mm
- net M3: track 361.8 -> 475.8 mm
- net ~RAS: track 235.1 -> 349.1 mm
- net M2: track 347.0 -> 461.0 mm
- net ~CAS: track 268.3 -> 382.3 mm
- net M5: track 356.1 -> 470.2 mm
- net M1: track 345.9 -> 460.0 mm
- net M0: track 345.9 -> 460.0 mm
- net ~VIRQ: track 0.00 -> 112.5 mm, vias 0 -> 1
- net -5V: track 452.0 -> 564.1 mm
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- added copper zone on F.Cu, net +5V

Commit message: 938 disconnected signals remain
Parts:
- moved C77 0.63 mm to (392.4, 207.0)
- moved R46 0.63 mm to (297.2, 231.1)
- moved R47 0.63 mm to (299.7, 231.1)
- moved R48 0.63 mm to (302.3, 231.1)
- moved R49 0.63 mm to (306.7, 231.1)
- moved REF** 0.63 mm to (176.5, 270.5)
Connections:
- RP5 pad 2: ~MRST -> PU1
- U100 pad 12: Net-(U100-Pad12) -> PU1
- U101 pad 3: Net-(U100-Pad12) -> PU1
- U67 pad 10: ~ODD1 -> ~EVEN1
- U67 pad 13: ~EVEN1 -> ~ODD1
- U67 pad 2: ~EVEN1 -> ~ODD1
- U67 pad 3: Net-(R36-Pad2) -> Net-(R21-Pad2)
- U67 pad 5: ~ODD1 -> ~EVEN1
- U67 pad 6: Net-(R21-Pad2) -> Net-(R36-Pad2)
- U79 pad 1: Net-(U67-Pad8) -> Net-(U67-Pad11)
- U80 pad 1: Net-(U67-Pad11) -> Net-(U67-Pad8)
Routing:
- net +5V: track 1464.4 -> 2401.9 mm
- net CCLK: track 0.00 -> 677.4 mm
- net ~E: track 0.00 -> 613.4 mm, vias 0 -> 1
- net Q: track 47.3 -> 656.0 mm, vias 1 -> 3
- net GND: track 1931.9 -> 2482.1 mm, vias 19 -> 23
- net ~EVEN0: track 7.62 -> 415.5 mm, vias 0 -> 2
- net ~ODD0: track 7.62 -> 401.5 mm, vias 0 -> 2
- net ~VRW: track 0.00 -> 363.0 mm, vias 0 -> 1
- net ~ODD1: track 7.62 -> 358.0 mm, vias 0 -> 2
- net ~EVEN1: track 7.62 -> 356.6 mm, vias 0 -> 2
- net ~MRST: track 78.5 -> 394.7 mm, vias 2 -> 4
- net R13: track 0.00 -> 299.6 mm, vias 0 -> 2
- net R14: track 5.08 -> 253.6 mm, vias 1 -> 3
- net -5V: track 564.1 -> 789.7 mm, vias 0 -> 2
- net +12V: track 558.6 -> 765.7 mm, vias 17 -> 21
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
Commit message: 792 disconnected signals remain
Parts:
- moved TP5 2.54 mm to (163.2, 241.3)
Routing:
- net GND: track 2482.1 -> 2669.4 mm, vias 23 -> 24
- net INV: track 4.44 -> 153.9 mm, vias 2 -> 3
- net BD1: track 0.00 -> 145.8 mm
- net ~5MHZ: track 37.7 -> 169.0 mm, vias 0 -> 1
- net VD5: track 70.1 -> 191.0 mm, vias 0 -> 1
- net _17: track 0.00 -> 119.4 mm, vias 0 -> 1
- net VD4: track 64.5 -> 181.4 mm, vias 0 -> 1
- net R6: track 0.00 -> 108.5 mm, vias 0 -> 2
- net R12: track 14.3 -> 115.7 mm, vias 1 -> 2
- net _16: track 0.00 -> 98.1 mm, vias 0 -> 1
- net S0: track 71.3 -> 169.1 mm
- net PR68: track 0.00 -> 97.8 mm
- net PR69: track 57.8 -> 155.5 mm
- net S1: track 69.4 -> 167.2 mm
- net VA1: track 68.0 -> 165.1 mm, vias 0 -> 2
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
Commit message: 694 disconnected signals remain
Connections:
- J6 pad 25: ~QX -> ~E
Routing:
- net ~VS3: track 23.1 -> 449.1 mm, vias 1 -> 4
- net R15: track 163.8 -> 467.1 mm, vias 2 -> 3
- net R31: track 0.00 -> 272.3 mm, vias 0 -> 2
- net R7: track 0.00 -> 203.0 mm, vias 0 -> 1
- net INV: track 153.9 -> 349.4 mm
- net ~RAS: track 349.1 -> 537.9 mm
- net R8: track 10.6 -> 175.1 mm, vias 1 -> 3
- net ~5MHZ: track 169.0 -> 311.1 mm, vias 1 -> 2
- net R23: track 0.00 -> 128.1 mm, vias 0 -> 1
- net Net-(R21-Pad1): track 0.00 -> 127.3 mm
- net GND: track 2669.4 -> 2792.8 mm, vias 24 -> 28
- net ~CAS: track 491.4 -> 605.5 mm
- net M6: track 471.4 -> 584.7 mm
- net M3: track 475.8 -> 587.5 mm
- net M0: track 460.0 -> 568.6 mm
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
Commit message: 578 disconnected signals remain
Parts:
- turned R53 to 270 degrees
Routing:
- net ~5MHZ: track 311.1 -> 447.1 mm, vias 2 -> 3
- net Net-(U40-Pad3): track 0.00 -> 107.4 mm, vias 0 -> 3
- net VD4: track 181.4 -> 287.4 mm, vias 1 -> 3
- net VD0: track 124.5 -> 230.2 mm, vias 3 -> 5
- net VD1: track 138.3 -> 240.1 mm, vias 1 -> 3
- net VD7: track 147.3 -> 242.5 mm
- net ~VS0: track 0.00 -> 91.1 mm, vias 0 -> 1
- net E: track 120.9 -> 211.5 mm, vias 1 -> 5
- net VD2: track 102.6 -> 189.1 mm, vias 2 -> 4
- net ~VRST: track 8.67 -> 93.2 mm, vias 0 -> 1
- net VD3: track 131.3 -> 212.7 mm, vias 1 -> 3
- net GND: track 2792.8 -> 2868.0 mm, vias 28 -> 32
- net ~INV: track 13.9 -> 83.7 mm, vias 1 -> 4
- net QX: track 0.00 -> 69.5 mm, vias 0 -> 1
- net ~E: track 694.5 -> 763.9 mm
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
Commit message: 540 disconnected signals remain
Routing:
- net R27: track 48.8 -> 208.9 mm
- net BD3: track 0.00 -> 145.9 mm
- net BD2: track 0.00 -> 145.9 mm
- net R16: track 15.4 -> 156.6 mm, vias 1 -> 2
- net R26: track 25.7 -> 159.7 mm, vias 2 -> 3
- net R25: track 12.9 -> 139.6 mm, vias 1 -> 2
- net R20: track 50.4 -> 167.4 mm, vias 2 -> 3
- net R18: track 31.9 -> 145.4 mm, vias 2 -> 3
- net M1: track 495.4 -> 607.1 mm
- net R21: track 16.3 -> 117.5 mm, vias 0 -> 1
- net R22: track 127.3 -> 219.1 mm, vias 2 -> 3
- net R17: track 34.8 -> 123.6 mm, vias 2 -> 3
- net R23: track 128.1 -> 216.3 mm, vias 1 -> 2
- net R24: track 120.7 -> 208.0 mm, vias 2 -> 3
- net ~RAS: track 537.9 -> 614.1 mm
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
Commit message: 490 disconnected signals remain
Routing:
- net R1: track 25.2 -> 231.8 mm, vias 2 -> 3
- net R28: track 51.3 -> 229.3 mm, vias 1 -> 2
- net R3: track 40.2 -> 212.8 mm, vias 2 -> 3
- net R2: track 12.9 -> 183.2 mm, vias 1 -> 2
- net VRW: track 132.7 -> 302.3 mm, vias 2 -> 5
- net ~VS6: track 0.00 -> 164.1 mm, vias 0 -> 3
- net ~VFIRQ: track 80.7 -> 234.5 mm, vias 1 -> 3
- net R30: track 99.9 -> 230.0 mm, vias 1 -> 3
- net ~VS0: track 91.1 -> 220.8 mm, vias 1 -> 2
- net R29: track 90.3 -> 215.3 mm
- net R31: track 272.3 -> 396.0 mm
- net ~VRST: track 93.2 -> 210.8 mm
- net M2: track 495.4 -> 604.0 mm
- net VE: track 59.7 -> 154.3 mm, vias 0 -> 1
- net VQ: track 64.6 -> 157.6 mm, vias 1 -> 2
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
Commit message: 467 disconnected signals remain
Routing:
- net R11: track 58.1 -> 303.4 mm
- net R10: track 93.4 -> 337.7 mm
- net R9: track 119.3 -> 320.9 mm
- net R6: track 108.5 -> 300.7 mm, vias 2 -> 5
- net R7: track 254.8 -> 418.3 mm
- net R5: track 99.2 -> 262.6 mm, vias 1 -> 3
- net BD5: track 0.00 -> 146.3 mm
- net R4: track 78.0 -> 208.6 mm, vias 4 -> 5
- net R0: track 116.2 -> 235.6 mm, vias 2 -> 3
- net R34: track 0.00 -> 38.9 mm
- net R2: track 183.2 -> 221.9 mm
- net R33: track 12.6 -> 48.7 mm
- net R50: track 35.3 -> 67.4 mm
- net R58: track 19.9 -> 50.8 mm, vias 1 -> 2
- net M4: track 582.1 -> 605.6 mm, vias 0 -> 1
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