File: taito_video_processor_pcb/taito_video_processor_pcb.kicad_pcb (KiCad board)
At the start: 2 copper layers, 304.8 x 279.4 mm, 352 parts, among them J1 14pin, J19 2pin, J2 14pin, J3 50pin, J6 50pin, Q1 2N3904, Q2 2N3904, Q3 2N3904, Q4 2N3904, Q5 2N3904, Q6 2N3904, Q7 2N3904, Q8 2N3905, SW1 SW_Push, U1 245_1, U10 4116, U100 LS00, U101 LS08, U102 LS10, U103 LS00, U104 157_1, U105 299_1, U106 299_1, U107 299_1, U108 299_1, U109 299_1, U11 4116, U110 299_1, U12 4116, U13 4116, U14 4116, U15 4116, U16 4116, U17 4116, U18 68A45, U19 86_2, U2 245_1, U20 86_1, U21 157_1, U22 LS32, U23 161_1, U24 LS04, U25 374_1, U26 4116, U27 4116, U28 4116, U29 4116, U3 2114, U30 4116, U31 4116, U32 4116, U33 4116, U34 LS374, U35 153_1, U36 LS74, U37 LS08, U38 74S113, U39 LS04, U4 2114, U40 7417, U41 4116, U42 4116, U43 4116, U44 4116, U45 4116, U46 4116, U47 4116, U48 4116, U49 LS32, U5 157_1, U50 86_3, U51 LS86, U52 153_1, U53 153_1, U54 153_1, U55 157_1, U56 2148_1, U57 2148_2, U58 7417, U59 4116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

Commit message: 409 disconnected signals remain
Routing:
- net R12: track 150.8 -> 437.8 mm, vias 3 -> 4
- net R8: track 191.0 -> 429.1 mm
- net CR4: track 20.2 -> 201.5 mm, vias 2 -> 3
- net CR5: track 25.4 -> 205.8 mm, vias 1 -> 2
- net CR7: track 17.0 -> 177.2 mm, vias 1 -> 2
- net CR6: track 25.2 -> 182.4 mm, vias 1 -> 2
- net Net-(FB4-Pad2): track 0.00 -> 150.0 mm
- net Net-(FB5-Pad2): track 0.00 -> 134.1 mm
- net R14: track 253.6 -> 380.2 mm
- net ~VEW: track 70.4 -> 196.4 mm, vias 1 -> 2
- net Net-(FB7-Pad1): track 0.00 -> 123.4 mm, vias 0 -> 1
- net Net-(FB6-Pad2): track 0.00 -> 117.1 mm, vias 0 -> 1
- net Net-(U49-Pad8): track 55.3 -> 168.8 mm
- net R44: track 20.2 -> 131.6 mm, vias 1 -> 2
- net R13: track 300.1 -> 411.5 mm
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
Commit message: 392 disconnected signals remain
Parts:
- moved R49 0.38 mm to (307.1, 231.1)
Routing:
- net Net-(FB7-Pad1): track 123.4 -> 277.9 mm, vias 1 -> 2
- net VEQ: track 152.2 -> 301.0 mm
- net BD6: track 4.44 -> 152.2 mm
- net BD7: track 0.00 -> 145.4 mm
- net ~INV: track 105.1 -> 250.1 mm, vias 5 -> 6
- net VRW: track 302.3 -> 401.0 mm, vias 5 -> 7
- net CR2: track 0.00 -> 94.5 mm, vias 0 -> 1
- net Net-(FB6-Pad2): track 117.1 -> 183.8 mm
- net R46: track 107.8 -> 155.2 mm
- net CR3: track 0.00 -> 47.1 mm, vias 0 -> 1
- net R3: track 241.9 -> 279.8 mm
- net VD0: track 230.2 -> 260.4 mm, vias 5 -> 6
- net M5: track 579.8 -> 604.9 mm, vias 0 -> 1
- net VD5: track 256.4 -> 276.5 mm, vias 3 -> 4
- net _00: track 84.8 -> 104.8 mm
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
Commit message: 300 disconnected signals remain
Routing:
- net INV: track 374.8 -> 578.3 mm
- net _VS: track 137.6 -> 322.7 mm, vias 0 -> 4
- net +5V: track 2503.9 -> 2634.4 mm, vias 1 -> 2
- net VD0: track 260.4 -> 378.1 mm
- net LA14: track 9.42 -> 122.7 mm
- net VD1: track 255.4 -> 367.0 mm
- net VD3: track 235.7 -> 341.4 mm, vias 4 -> 5
- net VD2: track 211.5 -> 316.5 mm
- net Net-(U103-Pad1): track 0.00 -> 96.2 mm, vias 0 -> 2
- net VD4: track 303.7 -> 397.7 mm
- net LA12: track 21.9 -> 112.1 mm
- net Net-(U19-Pad10): track 45.7 -> 135.8 mm
- net VD5: track 276.5 -> 365.1 mm
- net LA13: track 16.8 -> 104.6 mm
- net ~VEW: track 196.4 -> 284.2 mm
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
Commit message: 198 disconnected signal remain
Parts:
- moved Y1 0.51 mm to (265.9, 120.7)
Routing:
- net E: track 222.7 -> 418.5 mm, vias 5 -> 6
- net Net-(U103-Pad3): track 13.6 -> 159.8 mm
- net ~VS1: track 44.1 -> 187.9 mm, vias 1 -> 3
- net ~QRW: track 57.7 -> 195.0 mm
- net DA0: track 12.6 -> 149.7 mm, vias 1 -> 2
- net VD7: track 359.4 -> 485.7 mm, vias 3 -> 5
- net Net-(R61-Pad2): track 64.1 -> 183.7 mm
- net Net-(U102-Pad8): track 30.2 -> 142.5 mm, vias 1 -> 3
- net VD6: track 303.8 -> 414.8 mm, vias 3 -> 5
- net LA10: track 23.2 -> 132.9 mm
- net LA8: track 5.08 -> 114.6 mm
- net GND: track 3054.0 -> 3149.3 mm, vias 42 -> 43
- net CR1: track 54.4 -> 139.8 mm
- net AEN: track 61.2 -> 142.5 mm, vias 1 -> 2
- net LA12: track 112.1 -> 188.9 mm
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
Commit message: 97 disconnected signal remain
Routing:
- net VA9: track 111.7 -> 324.3 mm, vias 5 -> 6
- net VA8: track 110.0 -> 312.4 mm, vias 6 -> 7
- net VA2: track 104.4 -> 299.5 mm
- net VA5: track 113.1 -> 300.8 mm
- net VA4: track 115.9 -> 299.5 mm
- net VA3: track 115.7 -> 292.2 mm
- net VA7: track 146.6 -> 321.4 mm
- net ~VS7: track 0.00 -> 173.2 mm, vias 0 -> 1
- net VA6: track 145.4 -> 317.0 mm
- net VA0: track 222.7 -> 381.7 mm, vias 4 -> 5
- net VA1: track 165.1 -> 322.0 mm
- net ~VS4: track 85.3 -> 202.0 mm, vias 4 -> 5
- net VD7: track 485.7 -> 596.6 mm, vias 5 -> 6
- net LA5: track 10.7 -> 119.1 mm
- net ~INV: track 324.0 -> 418.4 mm, vias 9 -> 11
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
Commit message: PCB layout complete
Parts:
- added C999: .1uf, taito_video_processor_pcb:GenericComp, F.Cu at (253.4, 243.2)
Routing:
- net VEN: track 151.8 -> 325.2 mm
- net QX: track 111.3 -> 272.5 mm, vias 1 -> 5
- net Net-(U101-Pad6): track 28.7 -> 188.6 mm, vias 2 -> 3
- net VRW: track 462.5 -> 605.5 mm
- net Net-(FB3-Pad2): track 198.4 -> 328.8 mm, vias 2 -> 4
- net ~QX: track 61.5 -> 179.4 mm, vias 1 -> 2
- net M6: track 599.4 -> 706.4 mm
- net M5: track 604.9 -> 708.5 mm
- net VS: track 59.2 -> 162.0 mm
- net VA8: track 312.4 -> 414.5 mm
- net _VS: track 322.7 -> 424.6 mm
- net VA0: track 381.7 -> 483.3 mm
- net ~VFIRQ: track 251.0 -> 351.9 mm
- net HS: track 47.3 -> 146.3 mm
- net CCLK: track 733.8 -> 831.0 mm
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
Commit message: Restructured the project folders. Started the BOM
Parts:
- added G***: LOGO, Logo:Taito, F.Cu at (381.6, 346.1)
Other:
- board text added: "Designed By Nick Mikstas"

Commit message: Fixed upper left mounting hole and added CR2032 battery to PCB
Parts:
- added BT2: Battery_Cell, taito_video_processor_pcb:CR2032, F.Cu at (292.6, 342.9)
- added D1: FR156, taito_video_processor_pcb:GenericComp, F.Cu at (282.6, 332.1)
- R11, R12, R22, R23, R24, R25, R26, R27, R9: value ? -> 33
- moved REF** 1.42 mm to (160.0, 83.8)
Routing:
- net Net-(BT1-Pad1): track 11.1 -> 31.5 mm
- net Net-(BT1-Pad2): track 0.00 -> 14.0 mm
- net Net-(BT2-Pad1): track 0.00 -> 12.9 mm
- net ~ODD1: track 358.0 -> 357.4 mm
- net (no net): vias 0 -> 1
Other:
- board text added: "+"
- board text added: "-"
- board text added: "K"
